Commit message: Parte13 on going.

File: Parte12/p_ldalcol_description/urdf/p_ldalcol.urdf.xacro (robot description, xacro)
@@ -7,13 +7,13 @@
   <xacro:arg name="player_name" default="p_ldalcol" />
   <xacro:arg name="player_color" default="Blue" /> <!-- e.g. Red, Orange. Must exist in Gazebo/Colors and be defined in properties.xacro.-->
-  <!--Properties are global so they can be viewed from inside the included xacros-->
-  <!--  args are used with $(arg arg_name), properties are used as ${property_name}-->
-  <xacro:property name="player_name" value="$(arg player_name)"/>
-  <xacro:property name="player_color" value="$(arg player_color)"/>
+<!--  &lt;!&ndash;Properties are global so they can be viewed from inside the included xacros&ndash;&gt;-->
+<!--  &lt;!&ndash;  args are used with $(arg arg_name), properties are used as ${property_name}&ndash;&gt;-->
+<!--  <xacro:property name="player_name" value="$(arg player_name)"/>-->
+<!--  <xacro:property name="player_color" value="$(arg player_color)"/>-->
   <!-- Include other files-->
   <xacro:include filename="$(find p_ldalcol_description)/urdf/properties.xacro"/>
   <!--  <xacro:include filename="$(find ${player_name}_description)/urdf/player.gazebo.xacro"/>-->
   <xacro:include filename="$(find p_ldalcol_description)/urdf/p_ldalcol.gazebo.macro.xacro"/>
-  <xacro:gazebo_macro player_color="${player_color}" laser_visual="false" camera_visual="false" imu_visual="false"/>
+  <xacro:gazebo_macro player_color="$(arg player_color)" laser_visual="false" camera_visual="false" imu_visual="false"/>
   <link name="base_footprint"/>
   <joint name="base_joint" type="fixed">
@@ -28,5 +28,5 @@
         <mesh filename="package://turtlebot3_description/meshes/bases/waffle_pi_base.stl" scale="0.001 0.001 0.001"/>
       </geometry>
-      <material name="light_black"/>
+      <material name="$(arg player_color)"/>
     </visual>
     <collision>

File: Parte12/p_ldalcol_description/urdf/properties.xacro (robot description, xacro)
@@ -9,3 +9,12 @@
         <color rgba="1.0 0.4 0.0 1.0"/>
     </material>
+    <material name="Red">
+        <color rgba="1.0 0.0 0.0 1.0"/>
+    </material>
+    <material name="Green">
+        <color rgba="0.0 1.0 0.0 1.0"/>
+    </material>
+    <material name="Blue">
+        <color rgba="0.0 0.0 1.0 1.0"/>
+    </material>
 </robot>
