Commit message: Parte12 done.

File: Parte12/p_ldalcol_description/urdf/p_ldalcol.gazebo.macro.xacro (robot description, xacro)
@@ -1,9 +1,7 @@
 <?xml version="1.0"?>
-<robot name="p_ldalcol" xmlns:xacro="http://ros.org/wiki/xacro">
-  <xacro:arg name="laser_visual"  default="false"/>
-  <xacro:arg name="camera_visual" default="false"/>
-  <xacro:arg name="imu_visual"    default="false"/>
+<robot name="gazebo_macro" xmlns:xacro="http://ros.org/wiki/xacro">
+  <xacro:macro name="gazebo_macro" params="player_color laser_visual camera_visual imu_visual">
   <gazebo reference="base_link">
-    <material>Gazebo/White</material>
+    <material>Gazebo/${player_color}</material>
   </gazebo>
   <gazebo reference="wheel_left_link">
@@ -15,5 +13,5 @@
     <maxVel>0.1</maxVel>
     <fdir1>1 0 0</fdir1>
-    <material>Gazebo/Blue</material>
+    <material>Gazebo/FlatBlack</material>
   </gazebo>
   <gazebo reference="wheel_right_link">
@@ -25,5 +23,5 @@
     <maxVel>0.1</maxVel>
     <fdir1>1 0 0</fdir1>
-    <material>Gazebo/Blue</material>
+    <material>Gazebo/FlatBlack</material>
   </gazebo>
   <gazebo reference="caster_back_right_link">
@@ -34,5 +32,5 @@
     <minDepth>0.001</minDepth>
     <maxVel>1.0</maxVel>
-    <material>Gazebo/Blue</material>
+    <material>Gazebo/FlatBlack</material>
   </gazebo>
   <gazebo reference="caster_back_left_link">
@@ -43,12 +41,12 @@
     <minDepth>0.001</minDepth>
     <maxVel>1.0</maxVel>
-    <material>Gazebo/Blue</material>
+    <material>Gazebo/FlatBlack</material>
   </gazebo>
   <gazebo reference="imu_link">
     <sensor type="imu" name="imu">
       <always_on>true</always_on>
-      <visualize>$(arg imu_visual)</visualize>
+      <visualize>${imu_visual}</visualize>
     </sensor>
-    <material>Gazebo/White</material>
+    <material>Gazebo/Grey</material>
   </gazebo>
   <gazebo>
@@ -103,8 +101,8 @@
   </gazebo>
   <gazebo reference="base_scan">
-    <material>Gazebo/Blue</material>
+    <material>Gazebo/FlatBlack</material>
     <sensor type="ray" name="lds_lfcd_sensor">
       <pose>0 0 0 0 0 0</pose>
-      <visualize>$(arg laser_visual)</visualize>
+      <visualize>${laser_visual}</visualize>
       <update_rate>5</update_rate>
       <ray>
@@ -138,5 +136,5 @@
     <sensor type="camera" name="Pi Camera">
       <always_on>true</always_on>
-      <visualize>$(arg camera_visual)</visualize>
+      <visualize>${camera_visual}</visualize>
       <camera>
           <horizontal_fov>1.085595</horizontal_fov>
@@ -167,3 +165,4 @@
     </sensor>
   </gazebo>
+  </xacro:macro>
 </robot>

File: Parte12/p_ldalcol_description/urdf/p_ldalcol.urdf.xacro (robot description, xacro)
@@ -6,14 +6,14 @@
   <!--Args are local, properties are global, so we copy the values of the arguments to the properties-->
   <xacro:arg name="player_name" default="p_ldalcol" />
-<!--  <xacro:arg name="player_color" default="Blue" /> &lt;!&ndash; e.g. Red, Orange. Must exist in Gazebo/Colors and be defined in properties.xacro.&ndash;&gt;-->
+  <xacro:arg name="player_color" default="Blue" /> <!-- e.g. Red, Orange. Must exist in Gazebo/Colors and be defined in properties.xacro.-->
   <!--Properties are global so they can be viewed from inside the included xacros-->
   <!--  args are used with $(arg arg_name), properties are used as ${property_name}-->
   <xacro:property name="player_name" value="$(arg player_name)"/>
-<!--  <xacro:property name="player_color" value="$(arg player_color)"/>-->
+  <xacro:property name="player_color" value="$(arg player_color)"/>
   <!-- Include other files-->
   <xacro:include filename="$(find ${player_name}_description)/urdf/properties.xacro"/>
   <!--  <xacro:include filename="$(find ${player_name}_description)/urdf/player.gazebo.xacro"/>-->
-  <xacro:include filename="$(find ${player_name}_description)/urdf/p_ldalcol.gazebo.xacro"/>
-<!--  <xacro:gazebo_macro player_color="Blue" laser_visual="true" camera_visual="false" imu_visual="true"/>-->
+  <xacro:include filename="$(find ${player_name}_description)/urdf/p_ldalcol.gazebo.macro.xacro"/>
+  <xacro:gazebo_macro player_color="${player_color}" laser_visual="false" camera_visual="false" imu_visual="false"/>
   <link name="base_footprint"/>
   <joint name="base_joint" type="fixed">

Commit message: Adding the collision configuration.

File: Parte12/p_ldalcol_description/urdf/p_ldalcol.gazebo.macro.xacro (robot description, xacro)
@@ -4,4 +4,15 @@
   <gazebo reference="base_link">
     <material>Gazebo/${player_color}</material>
+    <sensor name="base_link" type="contact">
+      <update_rate>1000.0</update_rate>
+      <always_on>true</always_on>
+      <contact>
+        <collision>base_footprint_fixed_joint_lump__base_link_collision</collision>
+      </contact>
+      <plugin name="base_link_contact_sensor_plugin" filename="libgazebo_ros_bumper.so">
+        <bumperTopicName>contact</bumperTopicName>
+        <frameName>world</frameName>
+      </plugin>
+    </sensor>
   </gazebo>
   <gazebo reference="wheel_left_link">
